File: 01_PCB/Breadboard/Breadboard.kicad_sch (KiCad schematic)
At the start: 20 parts, among them J1 Screw_Terminal_01x02, J2 Screw_Terminal_01x02, J3 Screw_Terminal_01x03, J4 Screw_Terminal_01x03, J5 Screw_Terminal_01x03, J6 Screw_Terminal_01x03, J7 Conn_02x05_Odd_Even, J8 Screw_Terminal_01x03, J9 Screw_Terminal_01x03, Q1 IRF4905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

Commit message: Upload BOM
Parts:
- R1: value 560R -> 1K5
Changed lines of the file:
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@@
       (effects (font (size 1.27 1.27)) (justify left))
     )
-    (property "Value" "560R" (id 1) (at 67.31 67.3099 0)
+    (property "Value" "1K5" (id 1) (at 67.31 67.3099 0)
       (effects (font (size 1.27 1.27)) (justify left))
     )
@@
     )
     (path "/09d92a0c-2321-4447-ad0f-2be266ba9c13"
-      (reference "R1") (unit 1) (value "560R") (footprint "Resistor_THT:R_Axial_DIN0207_L6.3mm_D2.5mm_P7.62mm_Horizontal")
+      (reference "R1") (unit 1) (value "1K5") (footprint "Resistor_THT:R_Axial_DIN0207_L6.3mm_D2.5mm_P7.62mm_Horizontal")
     )
     (path "/787bdee5-46bf-4ed8-bd41-02fe61f05395"
